File: hardware/m749.kicad_sch (KiCad schematic)
At the start: 46 parts, among them J1_M74 502225-0801, U1 AT32F435ZMT7, U2 L9779WD-SPI, Y1 Resonator

Commit message: Add pdf file, update scheme.
Parts:
- added C? (x2): C_Small, symbol Device:C_Small
Connections:
- net +12V: now also J1_M74.2X/H1, J1_M74.2X/H2
- net GND: now also C?.2, C?.2, C?.2, C?.2, C?.2, C?.2, C?.2, C?.2, D?.2 (A), J1_M74.1X/D1, J1_M74.1X/E1, J1_M74.1X/F1, J1_M74.1X/G1, J1_M74.1X/H1, J1_M74.1X/H2, J1_M74.2X/C4, J1_M74.2X/D4, J1_M74.2X/G2, J1_M74.2X/G3, J1_M74.2X/G4, C?.2, C?.2
- net +5_VS2: now reaches U2.10 (VTRK2)
- net +5_VS2: now also J1_M74.1X/B4, J1_M74.2X/B4, C?.1
- net INJECTOR_2: now reaches U2.25 (OUT3)
- net INJECTOR_2: now also J1_M74.1X/G4
- net INJECTOR_1: now reaches U2.28 (OUT4)
- net INJECTOR_1: now also J1_M74.1X/F4
- net ADSORB_V: now reaches U2.57 (OUT5)
- net ADSORB_V: now also J1_M74.1X/E4
- net INJECTOR_4: now reaches U2.60 (OUT1)
- net INJECTOR_4: now also J1_M74.1X/J4
- net INJECTOR_3: now reaches U2.61 (OUT2)
- net INJECTOR_3: now also J1_M74.1X/H4
- net +5_VS1: now reaches U2.9 (VTRK1)
- net +5_VS1: now also J1_M74.1X/K1, J1_M74.2X/A4, C?.1
- net CRANK VR+: now reaches J1_M74.1X/A1
- net NC: now reaches J1_M74.1X/A2
- net NC: now also J1_M74.1X/A4, J1_M74.1X/B2, J1_M74.1X/C1, J1_M74.1X/G3, J1_M74.1X/L2, J1_M74.1X/L3, J1_M74.2X/E2, J1_M74.2X/H3
- net KNOCK+: now reaches J1_M74.1X/A3
- net CRANK VR-: now reaches J1_M74.1X/B1
- net KNOCK-: now reaches J1_M74.1X/B3
- net IAT: now reaches J1_M74.1X/C2
- net MAP: now reaches J1_M74.1X/C3
- net HEAT_OX_1: now reaches J1_M74.1X/C4
- net A/C: now reaches J1_M74.1X/D2
- net A/C: now also J1_M74.2X/D3
- net CTS: now reaches J1_M74.1X/D3
- net OIL_P_SW: now reaches J1_M74.1X/D4
- net CAN_L_2: now reaches J1_M74.1X/E2
- net CAN_H_2: now reaches J1_M74.1X/E3
- net SPEED IN: now reaches J1_M74.1X/F2
- net ALT DFM: now reaches J1_M74.1X/F3
- net CAM HAL: now reaches J1_M74.1X/G2
- net ALT_LT: now reaches J1_M74.1X/H3
- net TPS_ETC_2: now reaches J1_M74.1X/J2
- net IN_OX_2: now reaches J1_M74.1X/J3
- net TPS_ETC_1: now reaches J1_M74.1X/K2
- net IN_OX_1: now reaches J1_M74.1X/K3
- net HEAT_OX_2: now reaches J1_M74.1X/K4
- net IGN_1_(1-4): now reaches J1_M74.1X/L1
- net ETC-: now reaches J1_M74.1X/L4
- net IGN_3_(2-3): now reaches J1_M74.1X/M1
- net IGN_2: now reaches J1_M74.1X/M2
- net IGN_4: now reaches J1_M74.1X/M3
- net ETC+: now reaches J1_M74.1X/M4
- net A/C_RELAY: now reaches J1_M74.2X/A1
- net ACCEL_2: now reaches J1_M74.2X/A2
- net ACCEL_1: now reaches J1_M74.2X/A3
- net START_REL: now reaches J1_M74.2X/B1
- net AC_P(1-3): now reaches J1_M74.2X/B2
- net CLUTCH: now reaches J1_M74.2X/B3
- net FAN_REL_1: now reaches J1_M74.2X/C1
- net BRAKE_2: now reaches J1_M74.2X/C2
- net BRAKE_1: now reaches J1_M74.2X/C3
- net FAN_REL_2: now reaches J1_M74.2X/D1
- net CAN_L: now reaches J1_M74.2X/D2
- net MR: now reaches J1_M74.2X/E1
- net SPEED_OUT: now reaches J1_M74.2X/E3
- net CE_LAMP: now reaches J1_M74.2X/E4
- net CAN_H: now reaches J1_M74.2X/F1
- net IGN_KEY: now reaches J1_M74.2X/F2
- net AC_P(2): now reaches J1_M74.2X/F3
- net TAHO: now reaches J1_M74.2X/F4
- net FUEL_REL: now reaches J1_M74.2X/G1
- net FAN_FEED: now reaches J1_M74.2X/H4
- net not used: no longer names the net of C?.1, U2.4 (V3V3)
Other:
- note added: "not used"
- moved on the sheet: C?, R?

Commit message: update sheme
Parts:
- added C*1, C*2, C1, C18, C2, C26, C27, C3, C4, C6, C7: C_Small, symbol Device:C_Small
- added C*3: C*, symbol Device:C_Small
- added C23, C5: 100n, symbol Device:C_Small
- added D1, D7: NUP2105L, Package_TO_SOT_SMD:SOT-23, symbol Power_Protection:NUP2105L
- added D3: D_Small, symbol Device:D_Small
- added D6: DC_M3, Diode_SMD:D_SMB, symbol DC_Mx:DC_M3
- added J1: DAP_Conn_ARM_JTAG_SWD_10, symbol DAP_conn:DAP_Conn_ARM_JTAG_SWD_10
- added Q1, Q2, Q3, Q4: STGD18N40LZT4, Package_TO_SOT_SMD:TO-252-2, symbol IGBT:STGD18N40LZT4
- added R*1, R*2: R*, symbol Device:R_Small
- added R*3, R*4, R*5, R*6, R19: 0, symbol Device:R_Small
- added R1, R10, R2, R22, R3, R4, R7, R8, R9: R_Small, symbol Device:R_Small
- added R11, R12, R5, R6: 0*, symbol Device:R_Small
- added R13, R14: 10mOm, symbol Device:R_Small
- added R15, R16, R20, R21: 62, symbol Device:R_Small
- added R17: 1k, symbol Device:R_Small
- added U*1: TJA1042T ?*, Package_SO:SOIC-8_3.9x4.9mm_P1.27mm, symbol Interface_CAN_LIN:TJA1042T
- J1_M74: symbol molex_80pin:502225-0801 -> 502225-0801:502225-0801
- gave numbers to parts that had none: 40
- renumbered *C_ST to *C_ST1, *R_AT to *R_AT1, *R_ST to *R_ST1, *R_ST to *R_ST2
Connections:
- net +3.3V: now also C*3.2, J1.1 (VTref), R*1.2
- net +5V: now also C*1.1, C*2.1, U*1.3 (VCC)
- net CAN_H: now also U2.42 (CAN_H), D7.1 (K), R*5.2, R20.2
- net CAN_H_2: now also R*3.1, R*5.1
- net CAN_L: now also U2.41 (CAN_L), D7.2 (K), R*6.2, R21.2
- net CAN_L_2: now also R*4.1, R*6.1
- net GND: now also C*1.2, C*2.2, C*3.1, C1.1, C18.2, C2.1, C23.2, C26.2, C27.2, C3.1, C4.1, C5.2, C6.2, C7.2, D1.3 (A), D3.2 (A), D7.3 (A), J1.3 (GND), J1.5 (GND), J1.9 (GNDDetect), R1.2, R13.2, R14.2, R2.2, R22.2, R7.2, R8.2, U*1.2 (GND), U*1.8 (STB)
- net IGN_1_(1-4): now also C1.2, Q1.2 (C), R5.1
- net IGN_2: now also C3.2, Q3.2 (C), R11.1
- net IGN_3_(2-3): now also C2.2, Q2.2 (C), R6.1
- net IGN_4: now also C4.2, Q4.2 (C), R12.1
- net IGN_KEY: now also C6.1, R17.1
- net MR: now also D6.2 (A)
- net at C21.1, C24.1, Q5.1 (S)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: now also C26.1
- net DAP_2: now reaches U1.105 (PA13)
- net DAP_2: now also J1.2 (SWDIO/TMS)
- net DAP_4: now reaches U1.109 (PA14)
- net DAP_4: now also J1.4 (SWDCLK/TCK)
- net DAP_8: now reaches U1.110 (PA15)
- net DAP_8: now also J1.8 (--/TDI)
- net DAP_6: now reaches U1.133 (PB3)
- net DAP_6: now also J1.6 (--/TDO)
- net DAP_7: now reaches U1.134 (PB4)
- net DAP_7: now also J1.7 (NJTRST)
- net CAN_2_RX: now reaches U1.135 (PB5)
- net CAN_2_RX: now also U*1.4 (RXD)
- net CAN_2_TX: now reaches U1.136 (PB6)
- net CAN_2_TX: now also U*1.1 (TXD)
- net at U1.138 (BOOT0): now also C27.1, R22.1
- net DAP_10: now reaches U1.25 (NRST)
- net DAP_10: now also J1.10 (NRST)
- net CAN_RX: now reaches U1.56 (PG0)
- net CAN_RX: now also U2.43 (CAN_RX)
- net CAN_TX: now reaches U1.57 (PG1)
- net CAN_TX: now also U2.44 (CAN_TX)
- net at C11.1, C12.1, C14.1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: now also C18.1
- net at U2.11 (KEY_ON): now also R19.2
- net I_IGN_4: now reaches U2.14 (IGNI4)
- net I_IGN_3_(2-3): now reaches U2.15 (IGNI3)
- net I_IGN_2: now reaches U2.18 (IGNI2)
- net I_IGN_1_(1-4): now reaches U2.19 (IGNI1)
- net G_IGN_1_(1-4): now reaches U2.22 (IGN1)
- net G_IGN_1_(1-4): now also R1.1, R3.1
- net at U2.23 (MRD): now also D6.1 (K)
- net I_ADSORB_V: now reaches U2.35 (IN5)
- net I_INJECTOR_1: now reaches U2.36 (IN4)
- net I_INJECTOR_2: now reaches U2.37 (IN3)
- net I_INJECTOR_4: now reaches U2.39 (IN1)
- net I_INJECTOR_3: now reaches U2.48 (IN2)
- net G_IGN_2: now reaches U2.62 (IGN2)
- net G_IGN_2: now also R7.1, R9.1
- net G_IGN_3_(2-3): now reaches U2.63 (IGN3)
- net G_IGN_3_(2-3): now also R2.1, R4.1
- net G_IGN_4: now reaches U2.64 (IGN4)
- net G_IGN_4: now also R10.1, R8.1
- removed net NC: J1_M74.1X/A2, J1_M74.1X/A4, J1_M74.1X/B2, J1_M74.1X/C1, J1_M74.1X/G3, J1_M74.1X/L2, J1_M74.1X/L3, J1_M74.2X/E2, J1_M74.2X/H3
- new net: Q2.3 (E), Q4.3 (E), R14.1
- new net: C7.1, D3.1 (K), R17.2, R19.1
- new net: D1.2 (K), R*4.2, R16.2, U*1.6 (CANL)
- new net: Q1.1 (G), R3.2, R5.2
- new net: Q4.1 (G), R10.2, R12.2
- new net: C5.1, R*2.1, R15.1, R16.1
- new net: R*1.1, R*2.2, U*1.5 (SPLIT)
- new net: D1.1 (K), R*3.2, R15.2, U*1.7 (CANH)
- new net: C23.1, R20.1, R21.1
- new net: Q1.3 (E), Q3.3 (E), R13.1
- new net: Q3.1 (G), R11.2, R9.2
- new net: Q2.1 (G), R4.2, R6.2
Other:
- note added: "not soldered"
- moved on the sheet: C16, C21, C24, Q5, R18
