File: hardware/m749.kicad_sch (KiCad schematic)
At the start: 99 parts, among them J1 DAP_Conn_ARM_JTAG_SWD_10, J1_M74 502225-0801, Q1 STGD18N40LZT4, Q2 STGD18N40LZT4, Q3 STGD18N40LZT4, Q4 STGD18N40LZT4, Q5 STD20NF06, U1 AT32F435ZMT7, U2 L9779WD-SPI, U3 HT7533-1-SOT89, Y1 Resonator

Commit message: Update m749.kicad_sch
Parts:
- added C?: C_Small, symbol Device:C_Small
- added R?: 4.7k, symbol Device:R_Small
- added R? (x5): 10k, symbol Device:R_Small
Connections:
- net +3.3V: now also R?.1, R?.2, R?.2, R?.2, R?.2
- net +5V: now also C21.1, C24.1, C26.1, Q5.1 (S), U2.3 (VDD5)
- net DAP_10: now also C?.1, R?.2
- net DAP_2: now also R?.1
- net DAP_4: now also R?.2
- net DAP_6: now also R?.1
- net DAP_7: now also R?.1
- net DAP_8: now also R?.1
- net GND: now also C?.2, R?.1
- net HEAT_OX_1: now also U2.56 (OUT6)
- net HEAT_OX_2: now also U2.29 (OUT7)
- net I_ADSORB_V: now also U1.90 (PG5)
- net I_INJECTOR_1: now also U1.59 (PE8)
- net I_INJECTOR_2: now also U1.60 (PE9)
- net I_INJECTOR_3: now also U1.63 (PE10)
- net I_INJECTOR_4: now also U1.64 (PE11)
- net I_HEAT_OX_1: now reaches U1.91 (PG6)
- net I_HEAT_OX_1: now also U2.34 (IN6)
- net I_HEAT_OX_2: now reaches U1.92 (PG7)
- net I_HEAT_OX_2: now also U2.33 (IN7)
Other:
- moved on the sheet: C10, C11, C12, C14, C8, C9, D2, D4, R22

Commit message: Update m749.kicad_sch
Parts:
- added C? (x2): C_Small, symbol Device:C_Small
- added R? (x3): R_Small, symbol Device:R_Small
- added U? (x7): 74HC14, symbol 74xx:74HC14
Connections:
- net +5V: now also C?.1, R?.2, U?.14 (VCC)
- net CAM HAL: now also R?.1, R?.1
- net GND: now also C?.2, C?.2, U?.7 (GND)
- net CAMSHAFT: now reaches U1.140 (PB9)
- net CAMSHAFT: now also U?.4
- net CRANKSHAFT: now reaches U1.20 (PF8)
- net CRANKSHAFT: now also U?.2
- net VRS_OUT: now reaches U2.8 (OUT_VRS)
- net VRS_OUT: now also R?.1
- new net: R?.2, U?.1
- new net: C?.1, R?.2, U?.3

Commit message: Update m749.kicad_sch
Parts:
- added C?: C_Small, symbol Device:C_Small
- added R? (x3): R_Small, symbol Device:R_Small
Connections:
- net +5V: now also R?.2
- net ALT DFM: now also R?.1, R?.1, R?.2
- net GND: now also C?.2, R?.1
- net at U?.5: now also C?.1, R?.2
Other:
- moved on the sheet: C?, R?, U?B, U?C, U?D, U?E, U?F

Commit message: ADD TLE9201, ADD MUN5311, update sheme.
Parts:
- added C18, C22, C23, C29, C31: C_Small, symbol Device:C_Small
- added Q5: MUN5311DW1, symbol MUN5311DW1:MUN5311DW1
- added R20, R21, R22, R23: R_Small, symbol Device:R_Small
- added U3: TLE9201, symbol TLE9201:TLE9201
- gave numbers to parts that had none: 17
- renumbered C18 to C19, C19 to C20, C20 to C21, C21 to C24, C22 to C25, C23 to C26, C24 to C27, C25 to C28, C26 to C30, C27 to C36, C28 to C37, C29 to C38, C30 to C39, C31 to C40, C32 to C41, C33 to C42, C34 to C43, C35 to C44, C36 to C45, C37 to C46, C38 to C47, C39 to C48, C40 to C49, C41 to C50, C42 to C51, C43 to C52, C8 to C7, C7 to C8, J1_M74 to J1_M1, Q5 to Q6, R20 to R24, R21 to R25, R22 to R33, R23 to R34, R24 to R35, U3 to U1, U1 to U5
Connections:
- net +12V: now also C22.1, C23.1, U3.4 (VS)
- net +3.3V: now also C18.1, R23.1, U3.2 (VSO)
- net +5V: now also Q5.4 (E1), R20.2, R21.2
- net ETC+: now also C31.1, U3.5 (OUT1)
- net ETC-: now also C29.1, U3.7 (OUT2)
- net GND: now also C18.2, C22.2, C23.2, C29.2, C31.2, Q5.1 (E1), U3.6 (GND), U3.PAD
- net ETC_CS: now reaches U5.114 (PD0)
- net ETC_CS: now also R23.2, U3.9 (CSN)
- net ETC_SCK: now reaches U5.115 (PD1)
- net ETC_SCK: now also U3.10 (SCK)
- net ETC_SO: now reaches U5.117 (PD3)
- net ETC_SO: now also U3.3 (SO)
- net ETC_SI: now reaches U5.118 (PD4)
- net ETC_SI: now also U3.8 (SI)
- net ETC_PWM: now reaches U5.75 (PB14)
- net ETC_PWM: now also U3.12 (PWM)
- net ETC_DIR: now reaches U5.76 (PB15)
- net ETC_DIR: now also U3.1 (DIR)
- net ETC_WD: now reaches U2.38 (WDA)
- net ETC_WD: now also Q5.5 (B1), R20.1
- new net: Q5.6 (C1), R21.1, R22.1
- new net: Q5.3 (C1), R22.2, U3.11 (DIS)
- new net ETC_EN: Q5.2 (B1)

Commit message: Update m749.kicad_sch
partly ADC
Parts:
- added C? (x45): C_Small, symbol Device:C_Small
- added C? (x8): 1n, symbol Device:C_Small
- added D?: NUP2105L, Package_TO_SOT_SMD:SOT-23, symbol Power_Protection:NUP2105L
- added D?: BAT54SW, Package_TO_SOT_SMD:SOT-323_SC-70, symbol Diode:BAT54SW
- added D?: D_Small, symbol Device:D_Small
- added R*? (x2): 0, symbol Device:R_Small
- added R? (x22): 1k, symbol Device:R_Small
- added R? (x24): 22k, symbol Device:R_Small
- added R? (x2): R_Small, symbol Device:R_Small
- added R? (x2): 2.15k, symbol Device:R_Small
- added U? (x27): LMV358, symbol Amplifier_Operational:LMV358
Connections:
- net +3.3V: now also C?.1, C?.1, C?.1, C?.1, C?.1, C?.1, D?.2, R?.2, R?.2, R?.2, U?.8 (V+), U?.8 (V+), U?.8 (V+), U?.8 (V+), U?.8 (V+), U?.8 (V+)
- net +5V: now also C?.1, C?.1, C?.1, U?.8 (V+), U?.8 (V+), U?.8 (V+)
- net AC_P(1-3): now also R*?.1
- net ADSORB_V: now also C?.1
- net CTS: now also R?.1, R?.1
- net DAP_10: now also U2.5 (RST)
- net GND: now also C?.1, C?.2, C?.2, C?.2, C?.2, C?.2, C?.2, C?.2, C?.2, C?.2, C?.2, C?.2, C?.2, C?.2, C?.2, C?.2, C?.2, C?.2, C?.2, C?.2, C?.2, C?.2, C?.2, C?.2, C?.2, C?.2, C?.2, C?.2, C?.2, C?.2, C?.2, C?.2, C?.2, C?.2, C?.2, C?.2, C?.2, C?.2, C?.2, C?.2, C?.2, C?.2, C?.2, C?.2, C?.2, C?.2, C?.2, C?.2, C?.2, C?.2, C?.2, D?.1, D?.3 (A), R?.1, R?.1, R?.1, R?.1, R?.2, U?.4 (V-), U?.4 (V-), U?.4 (V-), U?.4 (V-), U?.4 (V-), U?.4 (V-), U?.4 (V-), U?.4 (V-), U?.4 (V-)
- net HEAT_OX_1: now also C?.1
- net HEAT_OX_2: now also C?.1
- net IAT: now also R?.1, R?.1
- net INJECTOR_1: now also C?.1
- net INJECTOR_2: now also C?.1
- net INJECTOR_3: now also C?.1
- net INJECTOR_4: now also C?.1
- net TAHO: now also R*?.1
- net at Q2.3 (E), Q4.3 (E), R14.1: now also R?.1
- net K_RX: now reaches U5.101 (PA9)
- net K_RX: now also R?.1, R?.1
- net K_TX: now reaches U5.102 (PA10)
- net K_TX: now also R?.1
- net I_ALT DFM: now reaches U5.111 (PC10)
- net I_ALT DFM: now also U4.6
- net at C36.1, R33.1, U5.138 (BOOT0): now also D?.3, R?.2
- net ADC_CTS: now reaches U5.15 (PF5)
- net ADC_CTS: now also C?.1, R?.2
- net ADC_IAT: now reaches U5.18 (PF6)
- net ADC_IAT: now also C?.1, R?.2
- net ADC_CUR_IG_1+2_(1-4): now reaches U5.46 (PB0)
- net ADC_CUR_IG_1+2_(1-4): now also C?.1, R?.2
- net ADC_CUR_IG_3+4_(2-3): now reaches U5.47 (PB1)
- net ADC_CUR_IG_3+4_(2-3): now also C?.1, R?.2
- net INTERNAL +12: now reaches C11.1, C12.1, C14.1, C16.1, C19.1, D4.1 (K), Q6.3 (D), U2.12 (VB)
- net INTERNAL +12: now also D?.2 (A)
- net at Q1.3 (E), Q3.3 (E), R13.1: now also R?.1
- net OUT_A: now reaches U2.13 (OUTA)
- net OUT_A: now also J1_M1.1X/L2
- net OUT_B: now reaches U2.16 (OUTB)
- net OUT_B: now also J1_M1.1X/L3
- net at U2.17 (OUTC): now also R*?.2
- net at U2.40 (OUT20): now also R*?.2
- net K_LINE: now reaches U2.45 (K_LINE)
- net K_LINE: now also J1_M1.1X/G3, C?.2, D?.2 (K), R?.1
- net at U2.46 (K_RX): now also R?.2
- net at U2.47 (K_TX): now also R?.2
- net _NOT_SOLDERED_OUTPUT_0: now reaches J1_M1.1X/A2
- net _ENABLE_REPROG: now reaches J1_M1.1X/A4
- net _ENABLE_REPROG: now also R?.1, R?.1
- net _NOT_SOLDERED_OUTPUT_1: now reaches J1_M1.1X/B2
- net _NOT_SOLDERED_ANALOG_INPUT_0: now reaches J1_M1.1X/C1
- net _NOT_SOLDERED_DISCRET_INPUT_0: now reaches J1_M1.1X/J1
- net _NOT_SOLDERED_OUTPUT_2: now reaches J1_M1.2X/E2
- net _NOT_SOLDERED_DISCRET_INPUT_1: now reaches J1_M1.2X/H3
- new net: R?.1, U?.6 (-), U?.7 (x8)
- new net: C?.1, R?.2 (x14)
- new net: C?.1, R?.1, R?.2, U?.6 (-)
- new net: C?.2, R?.1, R?.2, U?.7
- new net: C?.1, R?.2, U?.3 (+) (x8)
- new net: C?.1, R?.2, U?.5 (+) (x8)
- new net: R?.1, U?.1, U?.2 (-) (x8)
- new net: R?.2, R?.2, U?.5 (+)
- new net: R?.2, R?.2, U?.3 (+)
- new net: C?.2, R?.1, R?.2, U?.1
- new net: C?.1, R?.1, R?.2, U?.2 (-)
- new net: D?.1 (K), R?.2
Other:
- moved on the sheet: *C_ST1, *R_AT1, *R_ST1, *R_ST2, C*1, C*2, C*3, C1, C10, C11, C12, C13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
